File: uln/uln_0.02_backup.brd (EAGLE design)
At the start: 44.1 x 41.9 mm, 8 parts, among them IC1 ULN2003AD, IC2 74HC595D, IC3 ULN2003AD, J1 4P-2.0, J2 4P-2.0, J3 4P-2.0

Commit message: Updated uln2003 and l298 board
Last version ;)
Ready to be made at the hva lab
Parts:
- removed J3: 4P-2.0, Seeed-OPL-Connector:HW4-2.0
- moved JP1 71.5 mm to (0.00, -44.4)
- moved JP3 66.6 mm to (0.00, -63.2)
- moved J2 53.4 mm to (0.65, -28.0), turned to 0 degrees
- moved J1 29.2 mm to (0.65, -13.9), turned to 0 degrees
- moved IC1 15.3 mm to (10.2, 8.89), turned to 180 degrees
- moved IC2 13.1 mm to (10.2, 17.8), turned to 0 degrees
- moved IC3 10.6 mm to (21.6, 8.89), turned to 180 degrees
Connections:
- net N$11: now also J2.2; no longer J2.4
- net N$12: now also J2.1; no longer J1.1
- net N$13: now also J1.4; no longer J1.2
- net N$15: now also J1.2; no longer J1.4
- net N$16: now also IC3.10, J1.1; no longer IC3.14, J3.1
- net N$17: now also JP3.2; no longer JP3.3
- net N$18: now also JP3.3; no longer JP3.2
- net N$19: now also JP3.4; no longer JP3.1
- net N$8: now also IC3.7; no longer IC3.3
- net N$9: now also J2.4; no longer J2.2
- net VCC: now also JP3.1; no longer J2.1, JP3.4
Routing:
- added copper zone on layer 16, net N$20
Other:
- board outline removed
