File: uln/6 coils/uln_0.02.sch (EAGLE design)
At the start: 8 parts, among them IC1 ULN2003AD, IC2 74HC595D, IC3 ULN2003AD, J1 4P-2.0, J2 4P-2.0, J3 4P-2.0

Commit message: Updated uln2003 and l298 board
Last version ;)
Ready to be made at the hva lab
Parts:
- removed IC3: ULN2003AD, uln-udn:ULN2003AD
- removed J3: 4P-2.0, Seeed-OPL-Connector:GROVE-CONNECTOR-DIP(4P-2.0)
Connections:
- removed net N$16: IC3.O3, J3.1
- removed net N$8: IC2A.QA, IC3.I3
- net GND: no longer IC3.GND
- net VCC: no longer IC3.CD+
Changed lines of the file:
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@@
 </variantdefs>
 <classes>
-<class number="0" name="POWER" width="0.3048" drill="0.9906">
+<class number="0" name="POWER" width="0.3048" drill="0.0254">
 <clearance class="0" value="0.0254"/>
 </class>
-<class number="1" name="DATA" width="0.2032" drill="0.9906">
+<class number="1" name="DATA" width="0.2032" drill="0.0254">
 <clearance class="1" value="0.0254"/>
 </class>
@@
 <part name="JP1" library="SparkFun" deviceset="M03" device="PTH"/>
 <part name="JP3" library="SparkFun" deviceset="M04" device="PTH"/>
-<part name="IC3" library="uln-udn" deviceset="ULN2003A" device="D"/>
-<part name="GND1" library="SparkFun" deviceset="GND" device=""/>
-<part name="COILVOLTAGE1" library="SparkFun" deviceset="VCC" device="" value="COILVOLTAGE"/>
-<part name="J3" library="Seeed-OPL-Connector" deviceset="GROVE-CONNECTOR-DIP(4P-2.0)" device="" value="4P-2.0"/>
 </parts>
 <sheets>
@@
 <instance part="JP1" gate="G$1" x="-99.06" y="86.36"/>
 <instance part="JP3" gate="G$1" x="-78.74" y="63.5"/>
-<instance part="IC3" gate="A" x="55.88" y="101.6"/>
-<instance part="GND1" gate="1" x="40.64" y="91.44" rot="R270"/>
-<instance part="COILVOLTAGE1" gate="1" x="68.58" y="91.44" rot="R270"/>
-<instance part="J3" gate="G$1" x="105.41" y="100.33"/>
 </instances>
 <busses>
@@
 <wire x1="-91.44" y1="83.82" x2="-86.36" y2="83.82" width="0.1524" layer="91"/>
 </segment>
-<segment>
-<pinref part="IC3" gate="A" pin="GND"/>
-<pinref part="GND1" gate="1" pin="GND"/>
-</segment>
 </net>
 <net name="5V" class="1">
@@
 <pinref part="J2" gate="G$1" pin="1"/>
 <pinref part="P+1" gate="1" pin="VCC"/>
-</segment>
-<segment>
-<pinref part="IC3" gate="A" pin="CD+"/>
-<pinref part="COILVOLTAGE1" gate="1" pin="VCC"/>
 </segment>
 </net>
@@
 </segment>
 </net>
-<net name="N$8" class="1">
-<segment>
-<pinref part="IC2" gate="A" pin="QA"/>
-<wire x1="-2.54" y1="81.28" x2="27.94" y2="81.28" width="0.1524" layer="91"/>
-<wire x1="27.94" y1="81.28" x2="27.94" y2="93.98" width="0.1524" layer="91"/>
-<pinref part="IC3" gate="A" pin="I3"/>
-<wire x1="27.94" y1="93.98" x2="43.18" y2="104.14" width="0.1524" layer="91"/>
-</segment>
-</net>
-<net name="N$16" class="1">
-<segment>
-<pinref part="IC3" gate="A" pin="O3"/>
-<pinref part="J3" gate="G$1" pin="1"/>
-<wire x1="68.58" y1="104.14" x2="101.6" y2="104.14" width="0.1524" layer="91"/>
-</segment>
-</net>
