File: updated boards/uln_0.02.brd (EAGLE design)
At the start: 44.1 x 41.9 mm, 8 parts, among them IC1 ULN2003AD, IC2 74HC595D, IC3 ULN2003AD, J1 4P-2.0, J2 4P-2.0, J3 4P-2.0

Commit message: Updated uln2003 and l298 board
Last version ;)
Ready to be made at the hva lab
Routing:
- net N$8: track 0.00 -> 42.8 mm
- net VCC: track 0.00 -> 41.6 mm
- net GND: track 0.00 -> 37.0 mm
- net N$19: track 0.00 -> 29.5 mm
- net 5V: track 0.00 -> 24.2 mm, vias 0 -> 1
- net N$17: track 0.00 -> 18.7 mm
- net N$18: track 0.00 -> 18.2 mm, vias 0 -> 1
- net N$6: track 0.00 -> 17.2 mm, vias 0 -> 2
- net N$7: track 0.00 -> 12.5 mm, vias 0 -> 2
- net N$5: track 0.00 -> 11.1 mm
- net N$4: track 0.00 -> 11.1 mm
- net N$3: track 0.00 -> 11.1 mm
- net N$2: track 0.00 -> 11.1 mm
- net N$1: track 0.00 -> 10.8 mm
- net N$15: track 0.00 -> 10.2 mm
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Other:
- board size 44.1 x 41.9 mm -> 28.2 x 30.5 mm
